File: claire&mattPCB/cc_pcbRedo.kicad_sch (KiCad schematic)
At the start: 96 parts, among them J1 Conn_02x05_Odd_Even, J2 Micro_SD_Card_Det_Hirose_DM3AT, J3 4x4 Keypad, J4 DC-DC_JUMPER, J5 PS_WIRES, J6 PS_BJ, J7 DC-DC Converter, SW1 SW_Push, U1 ESP8266, U10 MAX7375AXR805, U2 7in_display_controller, U3 RFID_Scanner, U4 TFT_2.8IN_DISPLAY, U5 74HC14, U6 STM32F091RCTx, U7 MEZD71201AF, U8 TPS56325x, U9 4N28

Commit message: pcb finalization
Parts:
- J4: footprint Connector_PinSocket_1.27mm:PinSocket_2x03_P1.27mm_Vertical -> Connector_PinSocket_2.54mm:PinSocket_2x03_P2.54mm_Vertical
- J7: footprint imported_footprints:7.5Vdc-5Vdc_buck_converter -> (none)
Connections:
- net PC0: no longer U5.12
- net PC13: now also U5.12
Changed lines of the file:
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@@
     )
   )
-  (global_label "PC0" (shape input) (at 280.67 156.21 270) (fields_autoplaced)
+  (global_label "PC13" (shape input) (at 280.67 156.21 270) (fields_autoplaced)
     (effects (font (size 1.27 1.27)) (justify right))
-    (property "Intersheet References" "${INTERSHEET_REFS}" (id 0) (at 280.7494 162.3726 90)
+    (property "Intersheet References" "${INTERSHEET_REFS}" (id 0) (at 280.5906 163.5821 90)
       (effects (font (size 1.27 1.27)) (justify right) hide)
     )
@@
     (property "Reference" "J4" (id 0) (at 196.85 99.06 0))
     (property "Value" "DC-DC_JUMPER" (id 1) (at 196.85 101.6 0))
-    (property "Footprint" "Connector_PinSocket_1.27mm:PinSocket_2x03_P1.27mm_Vertical" (id 2) (at 195.58 107.95 0)
+    (property "Footprint" "Connector_PinSocket_2.54mm:PinSocket_2x03_P2.54mm_Vertical" (id 2) (at 195.58 107.95 0)
       (effects (font (size 1.27 1.27)) hide)
     )
@@
       (effects (font (size 1.27 1.27)) (justify left))
     )
-    (property "Footprint" "imported_footprints:7.5Vdc-5Vdc_buck_converter" (id 2) (at 204.47 67.31 0)
+    (property "Footprint" "" (id 2) (at 204.47 67.31 0)
       (effects (font (size 1.27 1.27)) hide)
     )
@@
       (effects (font (size 1.27 1.27)) hide)
     )
-    (property "Value" "" (id 1) (at 182.88 71.12 0))
+    (property "Value" "+5V" (id 1) (at 182.88 71.12 0))
     (property "Footprint" "" (id 2) (at 182.88 74.93 0)
       (effects (font (size 1.27 1.27)) hide)
@@
     )
     (path "/5302a90c-e22a-4144-afd8-6e77142a2010"
-      (reference "J4") (unit 1) (value "DC-DC_JUMPER") (footprint "Connector_PinSocket_1.27mm:PinSocket_2x03_P1.27mm_Vertical")
+      (reference "J4") (unit 1) (value "DC-DC_JUMPER") (footprint "Connector_PinSocket_2.54mm:PinSocket_2x03_P2.54mm_Vertical")
     )
     (path "/d6cf1125-b148-4911-9599-ed0399e2377f"
